Commit message: [ADD] prototype_v2.1.1]

File: prototype_v2.1.1/urdf/prototype_v2.1.1.urdf (robot description, URDF)
Before this commit: robot prototype_v2.1.1, 27 links, 26 joints
Links:
- added link left_foot_floor
- added link left_welding_point
- added link left_wrist_pitch_link, mass 0.20000000; collision mesh filename=../../prototype_v2.1/meshes/right_wrist_pitch_link.STL; visual mesh filename=../../prototype_v2.1/meshes/right_wrist_pitch_link.STL
- added link right_foot_floor
- added link right_welding_point
- added link right_wrist_pitch_link, mass 0.20000000; collision mesh filename=../../prototype_v2.1/meshes/right_wrist_pitch_link.STL; visual mesh filename=../../prototype_v2.1/meshes/right_wrist_pitch_link.STL
- link left_ankle_pitch_link: geometry collision mesh filename=../meshes/left_ankle_pitch_link.STL; visual mesh filename=../meshes/left_ankle_pitch_link.STL
- link left_ankle_roll_link: geometry collision mesh filename=../meshes/left_ankle_roll_link.STL; visual mesh filename=../meshes/left_ankle_roll_link.STL
- link left_elbow_pitch_link: geometry collision mesh filename=../meshes/left_elbow_pitch_link.STL; visual mesh filename=../meshes/left_elbow_pitch_link.STL
- link left_hip_pitch_link: geometry collision mesh filename=../meshes/left_hip_pitch_link.STL; visual mesh filename=../meshes/left_hip_pitch_link.STL
- link left_hip_roll_link: geometry collision mesh filename=../meshes/left_hip_roll_link.STL; visual mesh filename=../meshes/left_hip_roll_link.STL
- link left_hip_yaw_link: geometry collision mesh filename=../meshes/left_hip_yaw_link.STL; visual mesh filename=../meshes/left_hip_yaw_link.STL
- link left_knee_pitch_link: geometry collision mesh filename=../meshes/left_knee_pitch_link.STL; visual mesh filename=../meshes/left_knee_pitch_link.STL
- link left_shoulder_pitch_link: geometry collision mesh filename=../meshes/left_shoulder_pitch_link.STL; visual mesh filename=../meshes/left_shoulder_pitch_link.STL
- link left_shoulder_roll_link: geometry collision mesh filename=../meshes/left_shoulder_roll_link.STL; visual mesh filename=../meshes/left_shoulder_roll_link.STL
- link left_shoulder_yaw_link: geometry collision mesh filename=../meshes/left_shoulder_yaw_link.STL; visual mesh filename=../meshes/left_shoulder_yaw_link.STL
- link left_wrist_roll_link: geometry collision mesh filename=../meshes/left_wrist_roll_link.STL; visual mesh filename=../meshes/left_wrist_roll_link.STL
- link left_wrist_yaw_link: geometry collision mesh filename=../meshes/left_wrist_yaw_link.STL; visual mesh filename=../meshes/left_wrist_yaw_link.STL
- link pelvis_link: geometry collision mesh filename=../meshes/pelvis_link.STL; visual mesh filename=../meshes/pelvis_link.STL
- link right_ankle_pitch_link: geometry collision mesh filename=../meshes/right_ankle_pitch_link.STL; visual mesh filename=../meshes/right_ankle_pitch_link.STL
- link right_ankle_roll_link: geometry collision mesh filename=../meshes/right_ankle_roll_link.STL; visual mesh filename=../meshes/right_ankle_roll_link.STL
- link right_elbow_pitch_link: geometry collision mesh filename=../meshes/right_elbow_pitch_link.STL; visual mesh filename=../meshes/right_elbow_pitch_link.STL
- link right_hip_pitch_link: geometry collision mesh filename=../meshes/right_hip_pitch_link.STL; visual mesh filename=../meshes/right_hip_pitch_link.STL
- link right_hip_roll_link: geometry collision mesh filename=../meshes/right_hip_roll_link.STL; visual mesh filename=../meshes/right_hip_roll_link.STL
- link right_hip_yaw_link: geometry collision mesh filename=../meshes/right_hip_yaw_link.STL; visual mesh filename=../meshes/right_hip_yaw_link.STL
- link right_knee_pitch_link: geometry collision mesh filename=../meshes/right_knee_pitch_link.STL; visual mesh filename=../meshes/right_knee_pitch_link.STL
- link right_shoulder_pitch_link: geometry collision mesh filename=../meshes/right_shoulder_pitch_link.STL; visual mesh filename=../meshes/right_shoulder_pitch_link.STL
- link right_shoulder_roll_link: geometry collision mesh filename=../meshes/right_shoulder_roll_link.STL; visual mesh filename=../meshes/right_shoulder_roll_link.STL
- link right_shoulder_yaw_link: geometry collision mesh filename=../meshes/right_shoulder_yaw_link.STL; visual mesh filename=../meshes/right_shoulder_yaw_link.STL
- link right_wrist_roll_link: geometry collision mesh filename=../meshes/right_wrist_roll_link.STL; visual mesh filename=../meshes/right_wrist_roll_link.STL
- link right_wrist_yaw_link: geometry collision mesh filename=../meshes/right_wrist_yaw_link.STL; visual mesh filename=../meshes/right_wrist_yaw_link.STL
- link waist_pitch_link: geometry collision mesh filename=../meshes/waist_pitch_link.STL; visual mesh filename=../meshes/waist_pitch_link.STL
- link waist_yaw_link: geometry collision mesh filename=../meshes/waist_yaw_link.STL; visual mesh filename=../meshes/waist_yaw_link.STL
Joints:
- added joint left_foot_floor_joint: type fixed, parent left_ankle_roll_link, child left_foot_floor, origin xyz=-0.03225 0 -0.0735 rpy=0 0 0
- added joint left_welder_joint: type fixed, parent left_wrist_pitch_link, child left_welding_point, origin xyz=0.19535 -0.032 -0.01908 rpy=0 0 0
- added joint left_wrist_pitch_joint: type revolute, parent left_wrist_yaw_link, child left_wrist_pitch_link, origin xyz=0.097 0.0315 -0.0285 rpy=0 0 0, axis 0 1 0, limit lower=-1.570796 upper=1.570796 effort=36 velocity=11
- added joint right_foot_floor_joint: type fixed, parent right_ankle_roll_link, child right_foot_floor, origin xyz=-0.03225 0 -0.0735 rpy=0 0 0
- added joint right_welder_joint: type fixed, parent right_wrist_pitch_link, child right_welding_point, origin xyz=0.19535 -0.032 -0.01908 rpy=0 0 0
- added joint right_wrist_pitch_joint: type revolute, parent right_wrist_yaw_link, child right_wrist_pitch_link, origin xyz=0.097 0.0315 -0.0285 rpy=0 0 0, axis 0 1 0, limit lower=-1.570796 upper=1.570796 effort=36 velocity=11
- joint left_ankle_pitch_joint: limit lower=0 upper=0 effort=0 velocity=0 -> lower=-2.0944 upper=2.0944 effort=440 velocity=10
- joint left_ankle_roll_joint: limit lower=0 upper=0 effort=0 velocity=0 -> lower=-0.6981 upper=0.6981 effort=60 velocity=16
- joint left_elbow_pitch_joint: limit lower=0 upper=0 effort=0 velocity=0 -> lower=-0.698132 upper=3.839724 effort=120 velocity=16
- joint left_hip_pitch_joint: limit lower=0 upper=0 effort=0 velocity=0 -> lower=-3.1416 upper=3.1416 effort=440 velocity=10
- joint left_hip_roll_joint: limit lower=0 upper=0 effort=0 velocity=0 -> lower=-3.1416 upper=3.1416 effort=440 velocity=10
- joint left_hip_yaw_joint: limit lower=0 upper=0 effort=0 velocity=0 -> lower=-3.1416 upper=3.1416 effort=120 velocity=15
- joint left_knee_pitch_joint: limit lower=0 upper=0 effort=0 velocity=0 -> lower=-2.2689 upper=2.2689 effort=440 velocity=10
- joint left_shoulder_pitch_joint: limit lower=0 upper=0 effort=0 velocity=0 -> lower=-2.2252948 upper=2.2252948 effort=120 velocity=16
- joint left_shoulder_roll_joint: limit lower=0 upper=0 effort=0 velocity=0 -> lower=-0.261799 upper=3.403392 effort=120 velocity=16
- joint left_shoulder_yaw_joint: limit lower=0 upper=0 effort=0 velocity=0 -> lower=-2.225295 upper=2.225295 effort=120 velocity=16
- joint left_wrist_roll_joint: limit lower=0 upper=0 effort=0 velocity=0 -> lower=-2.967060 upper=2.967060 effort=60 velocity=18
- joint left_wrist_yaw_joint: limit lower=0 upper=0 effort=0 velocity=0 -> lower=-1.262747 upper=1.262747 effort=36 velocity=11
- joint right_ankle_pitch_joint: limit lower=0 upper=0 effort=0 velocity=0 -> lower=-2.0944 upper=2.0944 effort=440 velocity=10
- joint right_ankle_roll_joint: limit lower=0 upper=0 effort=0 velocity=0 -> lower=-0.6981 upper=0.6981 effort=60 velocity=16
- joint right_elbow_pitch_joint: limit lower=0 upper=0 effort=0 velocity=0 -> lower=-0.698132 upper=3.839724 effort=120 velocity=16
- joint right_hip_pitch_joint: limit lower=0 upper=0 effort=0 velocity=0 -> lower=-3.1416 upper=3.1416 effort=440 velocity=10
- joint right_hip_roll_joint: limit lower=0 upper=0 effort=0 velocity=0 -> lower=-3.1416 upper=3.1416 effort=440 velocity=10
- joint right_hip_yaw_joint: limit lower=0 upper=0 effort=0 velocity=0 -> lower=-3.1416 upper=3.1416 effort=120 velocity=15
- joint right_knee_pitch_joint: limit lower=0 upper=0 effort=0 velocity=0 -> lower=-2.2689 upper=2.2689 effort=440 velocity=10
- joint right_shoulder_pitch_joint: limit lower=0 upper=0 effort=0 velocity=0 -> lower=-2.2252948 upper=2.2252948 effort=120 velocity=16
- joint right_shoulder_roll_joint: limit lower=0 upper=0 effort=0 velocity=0 -> lower=-3.403392 upper=0.261799 effort=120 velocity=16
- joint right_shoulder_yaw_joint: limit lower=0 upper=0 effort=0 velocity=0 -> lower=-2.225295 upper=2.225295 effort=120 velocity=16
- joint right_wrist_roll_joint: limit lower=0 upper=0 effort=0 velocity=0 -> lower=-2.967060 upper=2.967060 effort=60 velocity=18
- joint right_wrist_yaw_joint: limit lower=0 upper=0 effort=0 velocity=0 -> lower=-1.262747 upper=1.262747 effort=36 velocity=11
- joint waist_pitch_joint: limit lower=0 upper=0 effort=0 velocity=0 -> lower=-0.5236 upper=1.5708 effort=880 velocity=10
- joint waist_yaw_joint: limit lower=0 upper=0 effort=0 velocity=0 -> lower=-3.1416 upper=3.1416 effort=120 velocity=15

Commit message: [ADD] robot spec test platform

File: prototype_v2.1.1/urdf/prototype_v2.1.1.urdf (robot description, URDF)
Before this commit: robot prototype_v2.1.1, 33 links, 32 joints
Links:
- link waist_pitch_link: mass 16.5953194153469 -> 32.23217336
